File: EsquemaKiCad/TK2000/TK2000.kicad_pcb (KiCad board)
At the start: 2 copper layers, 236.8 x 169.8 mm, 207 parts, among them J1 SolderJumper_2_Open, J10 SolderJumper_2_Open, J100 Joystick, J11 SolderJumper_2_Open, J12 SolderJumper_2_Open, J14 SolderJumper_2_Open, J16 SolderJumper_2_Open, J17 SolderJumper_2_Open_Small, J2 TK2000:Jumper_Open, J3 SolderJumper_2_Open, J4 SolderJumper_2_Open, J5 SolderJumper_2_Open, J6 SolderJumper_2_Open, J7 SolderJumper_2_Open, J8 SolderJumper_2_Open, J9 SolderJumper_2_Open, P1 POWER, P2 Conector de Expansão, P3 P3, P5 Conector_P5, Q1 BC548, Q2 BF494B, Q3 BC548, Q5 BC548, Q6 BC548, Q7 BC548, Q8 BD140, Q9 BD140, T2 MONITOR, T3 EAR, T4 MIC, T5 B - Remote, T6 A - Remote, T7 AUDIO, U10 74LS02, U11 74LS02, U12 74LS11, U13 74LS86, U14 74LS161, U15 74LS161, U16 74LS194, U17 74LS244, U18 74LS51, U19 74LS08, U2 74LS194, U20 74LS161, U21 74LS283, U22 74LS153, U23 74LS153, U24 74LS273, U25 74LS04, U26 74LS161, U27 74LS153, U28 74LS244, U29 6502, U3 74LS153, U30 74LS245, U31 LM741, U33 74LS32, U34 74LS153, U35 74LS244, U36 74LS259, U37 74LS74, U38 74LS138, U39 2764, U4 74LS175, U40 2764, U41 PAL14L4, U42 4116_U42, U43 4116_U43, U44 4116_U47, U45 4116_U47, U46 4116_U47, U47 4116_U47, U48 4116, U49 4116, U5 74LS04, U50 74LS138, U51 74LS174, U52 74LS157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

Commit message: Revisao 2: diodos em serie com R69/R71
Na placa original cada resistor de 5k6 (R69/R71) tem um diodo soldado
em serie. O footprint dos resistores passou para
Resistor_P5.08mm_Vertical e o lugar dos diodos foi incluido na PCB,
com a orientacao dos diodos corrigida.

- novo simbolo TK2000:D_Small e novo footprint TK2000:Diodo_5.715mm
- D69 e D71 (1N4148) adicionados em serie com R69 e R71
- arquivos de fabricacao da rev 2 (gerbers e BOM interativa)
- README da pasta Fabricacao
Parts:
- removed kibuzzard-66D4FA69: G***, kibuzzard-66D4FA69
- added D69: 1N4148, TK2000:Diodo_5.715mm, F.Cu at (117.7, 187.4)
- added D71: 1N4148, TK2000:Diodo_5.715mm, F.Cu at (117.4, 171.3)
- added kibuzzard-6AD42836: G***, kibuzzard-6AD42836, F.Cu at (252.7, 214.1)
- R69, R71: footprint TK2000:Resistor_P12.7mm_Horizontal -> TK2000:Resistor_P5.08mm_Vertical
- moved R71 7.62 mm to (117.4, 179.1)
- moved R69 7.41 mm to (117.7, 195.2)
Connections:
- R69 pad 1: Net-(U36-Q1) -> Net-(D69-A)
- R71 pad 1: Net-(U36-Q3) -> Net-(D71-A)
- U36 pad 5: Net-(U36-Q1) -> Net-(D69-K)
- U36 pad 7: Net-(U36-Q3) -> Net-(D71-K)
Routing:
- net Net-(U36-Q1): track 71.0 -> 0.00 mm, vias 2 -> 0
- net Net-(U36-Q3): track 71.0 -> 0.00 mm, vias 1 -> 0
- net Net-(D71-K): track 0.00 -> 71.0 mm, vias 0 -> 1
- net Net-(D69-K): track 0.00 -> 70.5 mm, vias 0 -> 2
- net Net-(D71-A): track 0.00 -> 2.08 mm
- net Net-(D69-A): track 0.00 -> 2.04 mm
