File: EsquemaKiCad/TK2000/extras.kicad_sch (KiCad schematic)
At the start: 48 parts, among them P1 POWER, P2 Conector de Expansão, T7 AUDIO, U10 74LS02, U11 74LS02, U12 74LS11, U13 74LS86, U18 74LS51, U19 74LS08, U25 74LS04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

Commit message: Finalização da Revisão 1
Other:
- company: Clemar Folly Jr. - https://www.x.com/clemarfolly -> Clemar Folly Jr. - https://www.x.com/clemarfolly - https://www.facebook.com/clemarjr
Changed lines of the file:
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@@
     (date "2024-08-30")
     (rev "1")
-    (company "Clemar Folly Jr. - https://www.x.com/clemarfolly")
+    (company "Clemar Folly Jr. - https://www.x.com/clemarfolly - https://www.facebook.com/clemarjr")
     (comment 1 "Recriado Por")
     (comment 2 "https://github.com/clemarfolly/Microdigital-TK2000")
